File: MOTHERBOARD/MOTHERBOARD.kicad_pcb (KiCad board)
At the start: 2 copper layers, 410 x 63 mm, 272 parts, among them J101 Conn_02x05_Odd_Even, J102 Conn_02x05_Odd_Even, J103 Conn_02x05_Odd_Even, J104 Conn_02x05_Odd_Even, J105 Conn_02x05_Odd_Even, J106 Conn_02x05_Odd_Even, J107 Conn_02x05_Odd_Even, J108 Conn_02x05_Odd_Even, J109 Conn_02x05_Odd_Even, J110 Conn_02x05_Odd_Even, J111 Conn_02x05_Odd_Even, J112 Conn_02x05_Odd_Even, J113 Conn_02x05_Odd_Even, J114 Conn_02x05_Odd_Even, J115 Conn_02x05_Odd_Even, J116 Conn_02x05_Odd_Even, J117 Conn_02x05_Odd_Even, J118 Conn_02x05_Odd_Even, J119 Conn_02x02_Odd_Even, Q301 MMBTA92, Q302 MMBTA92, Q303 MMBTA92, Q304 MMBTA92, Q401 MMBTA92, Q402 MMBTA92, Q403 MMBTA92, Q404 MMBTA92, Q501 MMBTA92, Q502 MMBTA92, Q503 MMBTA92, Q504 MMBTA92, Q601 MMBTA92, Q602 MMBTA92, Q603 MMBTA92, Q604 MMBTA92, U101 TL072, U301 TL074, U302 LM13700, U303 LM13700, U401 TL074, U402 LM13700, U403 LM13700, U501 TL074, U502 LM13700, U503 LM13700, U601 TL074, U602 LM13700, U603 LM13700

Commit message: Routed all the hard parts
Parts:
- moved D101 9.66 mm to (435.7, 279.4)
- moved R133 9.66 mm to (435.7, 284.8)
Routing:
- net -12V: track 741.0 -> 1089.9 mm, vias 31 -> 54
- net +12V: track 934.9 -> 1149.3 mm, vias 35 -> 44
- net /MOD_CARRIER_BANDS_LEFT: track 309.6 -> 407.0 mm, vias 8 -> 0
- net /MOD_CARRIER_BANDS_RIGHT: track 495.6 -> 525.9 mm, vias 7 -> 16
- net -2V: track 562.2 -> 568.9 mm
- net Net-(R509-Pad1): track 0.00 -> 3.07 mm
- net /CARRIER_BAND_16: track 27.5 -> 26.6 mm
- net /CARRIER_BAND_4: track 27.4 -> 26.7 mm
- net /PROGRAM_ENV_16: track 53.6 -> 53.0 mm
- net /CARRIER_BAND_12: track 27.3 -> 26.7 mm
Other:
- board text added: "Theory tells us that electronics, such as microchips, are secretly powered using hidden scientific laws one might describe as more akin to “magic” than to “science”. The secretive few who know the true properties of modern electronics want to keep us in the dark in order to continue their control over us using these devices. Ask yourself which of the following statements ring true: There are bill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"

Commit message: New series resistor values for LEDs
Parts:
- removed R133: 470, Resistor_SMD:R_0603_1608Metric_Pad0.98x0.95mm_HandSolder
Routing:
- net Net-(D101-Pad1): track 4.54 -> 0.00 mm
