File: POWERBOARD/POWERBOARD.kicad_pcb (KiCad board)
At the start: 2 copper layers, 120 x 60 mm, 25 parts, among them J201 Conn_01x02_Female, J202 Conn_02x02_Odd_Even, T201 VPP36-140, U201 uA7812, U202 uA7912

Commit message: Initial commit
Routing:
- net Net-(D201-Pad2): track 57.7 -> 61.1 mm
- net Net-(D202-Pad2): track 53.4 -> 56.7 mm
